Commit message: added red car model to Rviz without any transform

File: racecar_blue.xacro (robot description, xacro)
@@ -1,5 +1,5 @@
 <?xml version="1.0"?>
 <!-- A simple model of the racecar for rviz -->
-<robot xmlns:xacro="http://www.ros.org/wiki/xacro" name="racecar1">
+<robot xmlns:xacro="http://www.ros.org/wiki/xacro" name="racecar_blue">
   <xacro:property name="wheelbase" value="0.3302" />
   <xacro:property name="width" value="0.2032" />
@@ -17,5 +17,7 @@
     <color rgba="0.3 0.57 1. 1."/>
   </material>
-  <link name="base_link">
+  <!-- added blue/ to all name -->
+  <!-- also need to add blue/ to params.yaml and simulator.cpp where mentioned frame of blue car -->
+  <link name="blue/base_link">
     <visual>
       <origin xyz="${wheelbase/2} 0 ${ground_offset+height/2}"/>
@@ -27,9 +29,9 @@
   </link>
   <joint name="base_to_laser_model" type="fixed">
-    <parent link="base_link"/>
-    <child link="laser_model"/>
+    <parent link="blue/base_link"/>
+    <child link="blue/laser_model"/>
     <origin xyz="${laser_distance_from_base_link} 0 ${ground_offset+height+(laser_height/2)}"/>
   </joint>
-  <link name="laser_model">
+  <link name="blue/laser_model">
     <visual>
       <geometry>
@@ -39,10 +41,10 @@
     </visual>
   </link>
-  <joint name="base_to_back_left_wheel" type="fixed">
-    <parent link="base_link"/>
-    <child link="back_left_wheel"/>
+  <joint name="blue/base_to_back_left_wheel" type="fixed">
+    <parent link="blue/base_link"/>
+    <child link="blue/back_left_wheel"/>
     <origin xyz="0 ${(wheel_length+width)/2} ${wheel_radius}"/>
   </joint>
-  <link name="back_left_wheel">
+  <link name="blue/back_left_wheel">
     <visual>
       <geometry>
@@ -53,10 +55,10 @@
     </visual>
   </link>
-  <joint name="base_to_back_right_wheel" type="fixed">
-    <parent link="base_link"/>
-    <child link="back_right_wheel"/>
+  <joint name="blue/base_to_back_right_wheel" type="fixed">
+    <parent link="blue/base_link"/>
+    <child link="blue/back_right_wheel"/>
     <origin xyz="0 ${-(wheel_length+width)/2} ${wheel_radius}"/>
   </joint>
-  <link name="back_right_wheel">
+  <link name="blue/back_right_wheel">
     <visual>
       <geometry>
@@ -67,15 +69,15 @@
     </visual>
   </link>
-  <joint name="base_to_front_left_hinge" type="fixed">
-    <parent link="base_link"/>
-    <child link="front_left_hinge"/>
+  <joint name="blue/base_to_front_left_hinge" type="fixed">
+    <parent link="blue/base_link"/>
+    <child link="blue/front_left_hinge"/>
     <origin xyz="${wheelbase} ${(wheel_length+width)/2} ${wheel_radius}"/>
   </joint>
-  <link name="front_left_hinge"/>
-  <joint name="front_left_hinge_to_wheel" type="continuous">
-    <parent link="front_left_hinge"/>
-    <child link="front_left_wheel"/>
+  <link name="blue/front_left_hinge"/>
+  <joint name="blue/front_left_hinge_to_wheel" type="continuous">
+    <parent link="blue/front_left_hinge"/>
+    <child link="blue/front_left_wheel"/>
   </joint>
-  <link name="front_left_wheel">
+  <link name="blue/front_left_wheel">
     <visual>
       <geometry>
@@ -86,15 +88,15 @@
     </visual>
   </link>
-  <joint name="base_to_front_right_hinge" type="fixed">
-    <parent link="base_link"/>
-    <child link="front_right_hinge"/>
+  <joint name="blue/base_to_front_right_hinge" type="fixed">
+    <parent link="blue/base_link"/>
+    <child link="blue/front_right_hinge"/>
     <origin xyz="${wheelbase} ${-(wheel_length+width)/2} ${wheel_radius}"/>
   </joint>
-  <link name="front_right_hinge"/>
-  <joint name="front_right_hinge_to_wheel" type="continuous">
-    <parent link="front_right_hinge"/>
-    <child link="front_right_wheel"/>
+  <link name="blue/front_right_hinge"/>
+  <joint name="blue/front_right_hinge_to_wheel" type="continuous">
+    <parent link="blue/front_right_hinge"/>
+    <child link="blue/front_right_wheel"/>
   </joint>
-  <link name="front_right_wheel">
+  <link name="blue/front_right_wheel">
     <visual>
       <geometry>

File: racecar_red.xacro (robot description, xacro)
@@ -1,5 +1,5 @@
 <?xml version="1.0"?>
 <!-- A simple model of the racecar for rviz -->
-<robot xmlns:xacro="http://www.ros.org/wiki/xacro" name="racecar">
+<robot xmlns:xacro="http://www.ros.org/wiki/xacro" name="racecar_red">
   <xacro:property name="wheelbase" value="0.3302" />
   <xacro:property name="width" value="0.2032" />
@@ -14,6 +14,6 @@
     <color rgba="0.2 0.2 0.2 1."/>
   </material>
-  <material name="blue">
-    <color rgba="0.3 0.57 1. 1."/>
+  <material name="red">
+    <color rgba="1 0.57 0.3 1."/>
   </material>
   <link name="base_link">
@@ -23,5 +23,5 @@
         <box size="${wheelbase} ${width} ${height}"/>
       </geometry>
-      <material name="blue"/>
+      <material name="red"/>
     </visual>
   </link>
