Commit message: almost make two car can be controlled by keyboard

File: racecar_red.xacro (robot description, xacro)
@@ -17,5 +17,5 @@
     <color rgba="1 0.57 0.3 1."/>
   </material>
-  <link name="base_link">
+  <link name="red/base_link">
     <visual>
       <origin xyz="${wheelbase/2} 0 ${ground_offset+height/2}"/>
@@ -27,9 +27,9 @@
   </link>
   <joint name="base_to_laser_model" type="fixed">
-    <parent link="base_link"/>
-    <child link="laser_model"/>
+    <parent link="red/base_link"/>
+    <child link="red/laser_model"/>
     <origin xyz="${laser_distance_from_base_link} 0 ${ground_offset+height+(laser_height/2)}"/>
   </joint>
-  <link name="laser_model">
+  <link name="red/laser_model">
     <visual>
       <geometry>
@@ -39,10 +39,10 @@
     </visual>
   </link>
-  <joint name="base_to_back_left_wheel" type="fixed">
-    <parent link="base_link"/>
-    <child link="back_left_wheel"/>
+  <joint name="red/base_to_back_left_wheel" type="fixed">
+    <parent link="red/base_link"/>
+    <child link="red/back_left_wheel"/>
     <origin xyz="0 ${(wheel_length+width)/2} ${wheel_radius}"/>
   </joint>
-  <link name="back_left_wheel">
+  <link name="red/back_left_wheel">
     <visual>
       <geometry>
@@ -53,10 +53,10 @@
     </visual>
   </link>
-  <joint name="base_to_back_right_wheel" type="fixed">
-    <parent link="base_link"/>
-    <child link="back_right_wheel"/>
+  <joint name="red/base_to_back_right_wheel" type="fixed">
+    <parent link="red/base_link"/>
+    <child link="red/back_right_wheel"/>
     <origin xyz="0 ${-(wheel_length+width)/2} ${wheel_radius}"/>
   </joint>
-  <link name="back_right_wheel">
+  <link name="red/back_right_wheel">
     <visual>
       <geometry>
@@ -67,15 +67,15 @@
     </visual>
   </link>
-  <joint name="base_to_front_left_hinge" type="fixed">
-    <parent link="base_link"/>
-    <child link="front_left_hinge"/>
+  <joint name="red/base_to_front_left_hinge" type="fixed">
+    <parent link="red/base_link"/>
+    <child link="red/front_left_hinge"/>
     <origin xyz="${wheelbase} ${(wheel_length+width)/2} ${wheel_radius}"/>
   </joint>
-  <link name="front_left_hinge"/>
-  <joint name="front_left_hinge_to_wheel" type="continuous">
-    <parent link="front_left_hinge"/>
-    <child link="front_left_wheel"/>
+  <link name="red/front_left_hinge"/>
+  <joint name="red/front_left_hinge_to_wheel" type="continuous">
+    <parent link="red/front_left_hinge"/>
+    <child link="red/front_left_wheel"/>
   </joint>
-  <link name="front_left_wheel">
+  <link name="red/front_left_wheel">
     <visual>
       <geometry>
@@ -86,15 +86,15 @@
     </visual>
   </link>
-  <joint name="base_to_front_right_hinge" type="fixed">
-    <parent link="base_link"/>
-    <child link="front_right_hinge"/>
+  <joint name="red/base_to_front_right_hinge" type="fixed">
+    <parent link="red/base_link"/>
+    <child link="red/front_right_hinge"/>
     <origin xyz="${wheelbase} ${-(wheel_length+width)/2} ${wheel_radius}"/>
   </joint>
-  <link name="front_right_hinge"/>
-  <joint name="front_right_hinge_to_wheel" type="continuous">
-    <parent link="front_right_hinge"/>
-    <child link="front_right_wheel"/>
+  <link name="red/front_right_hinge"/>
+  <joint name="red/front_right_hinge_to_wheel" type="continuous">
+    <parent link="red/front_right_hinge"/>
+    <child link="red/front_right_wheel"/>
   </joint>
-  <link name="front_right_wheel">
+  <link name="red/front_right_wheel">
     <visual>
       <geometry>
